Commit message: added SLAM

File: description/lidar.xacro (robot description, xacro)
@@ -38,5 +38,5 @@
                 <range>
                     <min>0.3</min>
-                    <max>12</max>
+                    <max>20</max>
                 </range>
             </ray>

File: description/robot_core.xacro (robot description, xacro)
@@ -20,4 +20,11 @@
 	<link name="base_link">
 	</link>
+	<!-- BASE_FOOTPRINT LINK -->
+	<joint name="base_footprint_joint" type="fixed">
+		<parent link="base_link"/>
+		<child link="base_footprint"/>
+		<origin xyz="0 0 0" rpy="0 0 0"/>
+	</joint>
+	<link name="base_footprint"></link>
 	<!-- CHASSIS LINK -->
 	<joint name="chassis_joint" type="fixed">
